File: kicad-egyoldalas/pico-gps-spedometer.kicad_sch (KiCad schematic)
At the start: 21 parts, among them J1 Akkumulátor be, J2 TP4056-18650-Charger, J3 uBlox NEO GPS (6M/8M), Q1 PN2222A, U1 RP2040-ZERO, U2 DS18B20, U3 LM7805_TO220, U4 TFT_320x240

Commit message: Refactor code structure for improved readability and maintainability
Parts:
- R5: footprint Connector_PinHeader_2.54mm:PinHeader_1x02_P2.54mm_Vertical -> OptoDevice:R_LDR_4.9x4.2mm_P2.54mm_Vertical
- U2: footprint Connector_PinHeader_2.54mm:PinHeader_1x03_P2.54mm_Vertical -> Package_TO_SOT_THT:TO-92_Inline
Changed lines of the file:
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@@
 			)
 		)
-		(property "Footprint" "Connector_PinHeader_2.54mm:PinHeader_1x03_P2.54mm_Vertical"
+		(property "Footprint" "Package_TO_SOT_THT:TO-92_Inline"
 			(at 21.59 115.57 0)
 			(effects
@@
 			)
 		)
-		(property "Footprint" "Connector_PinHeader_2.54mm:PinHeader_1x02_P2.54mm_Vertical"
+		(property "Footprint" "OptoDevice:R_LDR_4.9x4.2mm_P2.54mm_Vertical"
 			(at 168.91 97.79 90)
 			(effects
