File: kicad.old/pico-gps-spedometer.kicad_pcb (KiCad board)
At the start: 2 copper layers, 89 x 76 mm, 32 parts, among them J1 Akkumulátor be, J2 TP4056-18650-Charger, J3 uBlox NEO GPS (6M/8M), Q1 PN2222A, Q2 PN2222A, U1 RP2040-ZERO, U2 DS18B20, U3 LM7805_TO220, U4 TFT_320x240

Commit message: Refactor code structure and remove redundant sections for improved readability and maintainability
Parts:
- R9: footprint Resistor_THT:R_Axial_DIN0204_L3.6mm_D1.6mm_P7.62mm_Horizontal -> Resistor_THT:R_Axial_DIN0207_L6.3mm_D2.5mm_P10.16mm_Horizontal
- moved R9 31.1 mm to (60.5, 31.3), turned to -90 degrees
- moved R10 28.8 mm to (60.5, 43.8), turned to -90 degrees
Routing:
- net /MISO: track 63.2 -> 28.2 mm
- net Net-(U1-GP28): track 0.00 -> 11.5 mm
- net +BATT: track 141.5 -> 149.8 mm
- net GND: track 343.4 -> 346.6 mm
- net /T_CS: track 52.5 -> 51.1 mm
- net /SCK: track 42.6 -> 41.9 mm
