File: kicad.old/pico-gps-spedometer.kicad_sch (KiCad schematic)
At the start: 26 parts, among them J1 Akkumulátor be, J2 TP4056-18650-Charger, J3 uBlox NEO GPS (6M/8M), Q1 PN2222A, Q2 PN2222A, U1 RP2040-ZERO, U2 DS18B20, U3 LM7805_TO220, U4 TFT_320x240

Commit message: Refactor code structure and remove redundant sections for improved readability and maintainability
Parts:
- R9: footprint Resistor_THT:R_Axial_DIN0204_L3.6mm_D1.6mm_P7.62mm_Horizontal -> Resistor_THT:R_Axial_DIN0207_L6.3mm_D2.5mm_P10.16mm_Horizontal
Other:
- moved on the sheet: R10, R3, R6
Changed lines of the file:
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@@
 	(wire
 		(pts
-			(xy 166.37 104.14) (xy 166.37 109.22)
+			(xy 166.37 104.14) (xy 166.37 110.49)
 		)
 		(stroke
@@
 	(wire
 		(pts
+			(xy 154.94 110.49) (xy 154.94 109.22)
+		)
+		(stroke
+			(width 0)
+			(type default)
+		)
+	)
+	(wire
+		(pts
 			(xy 138.43 36.83) (xy 143.51 36.83)
 		)
@@
 	(wire
 		(pts
-			(xy 154.94 116.84) (xy 154.94 120.65)
+			(xy 154.94 118.11) (xy 154.94 120.65)
 		)
 		(stroke
@@
 	(wire
 		(pts
-			(xy 179.07 106.68) (xy 179.07 109.22)
+			(xy 179.07 106.68) (xy 179.07 110.49)
 		)
 		(stroke
@@
 	(wire
 		(pts
-			(xy 179.07 116.84) (xy 179.07 120.65)
+			(xy 179.07 118.11) (xy 179.07 120.65)
 		)
 		(stroke
@@
 	(wire
 		(pts
-			(xy 166.37 116.84) (xy 166.37 120.65)
+			(xy 166.37 118.11) (xy 166.37 120.65)
 		)
 		(stroke
@@
 			)
 		)
-		(property "Footprint" "Resistor_THT:R_Axial_DIN0204_L3.6mm_D1.6mm_P7.62mm_Horizontal"
+		(property "Footprint" "Resistor_THT:R_Axial_DIN0207_L6.3mm_D2.5mm_P10.16mm_Horizontal"
 			(at 153.162 91.44 90)
 			(effects
@@
 	(symbol
 		(lib_id "Device:R")
-		(at 154.94 113.03 0)
+		(at 154.94 114.3 0)
 		(unit 1)
 		(exclude_from_sim no)
@@
 		(fields_autoplaced yes)
 		(property "Reference" "R10"
-			(at 157.48 111.7599 0)
+			(at 157.48 113.0299 0)
 			(effects
 				(font
@@
 		)
 		(property "Value" "10k"
-			(at 157.48 114.2999 0)
+			(at 157.48 115.5699 0)
 			(effects
 				(font
@@
 		)
 		(property "Footprint" "Resistor_THT:R_Axial_DIN0204_L3.6mm_D1.6mm_P7.62mm_Horizontal"
-			(at 153.162 113.03 90)
+			(at 153.162 114.3 90)
 			(effects
 				(font
@@
 		)
 		(property "Datasheet" "~"
-			(at 154.94 113.03 0)
+			(at 154.94 114.3 0)
 			(effects
 				(font
@@
 		)
 		(property "Description" "Resistor"
-			(at 154.94 113.03 0)
+			(at 154.94 114.3 0)
 			(effects
 				(font
@@
 	(symbol
 		(lib_id "Device:R")
-		(at 179.07 113.03 0)
+		(at 179.07 114.3 0)
 		(unit 1)
 		(exclude_from_sim no)
@@
 		(fields_autoplaced yes)
 		(property "Reference" "R6"
-			(at 181.61 111.7599 0)
+			(at 181.61 113.0299 0)
 			(effects
 				(font
@@
 		)
 		(property "Value" "10k"
-			(at 181.61 114.2999 0)
+			(at 181.61 115.5699 0)
 			(effects
 				(font
@@
 		)
 		(property "Footprint" "Resistor_THT:R_Axial_DIN0204_L3.6mm_D1.6mm_P7.62mm_Horizontal"
-			(at 177.292 113.03 90)
+			(at 177.292 114.3 90)
 			(effects
 				(font
@@
 		)
 		(property "Datasheet" "~"
-			(at 179.07 113.03 0)
+			(at 179.07 114.3 0)
 			(effects
 				(font
@@
 		)
 		(property "Description" "Resistor"
-			(at 179.07 113.03 0)
+			(at 179.07 114.3 0)
 			(effects
 				(font
@@
 	(symbol
 		(lib_id "Device:R")
-		(at 166.37 113.03 0)
+		(at 166.37 114.3 0)
 		(unit 1)
 		(exclude_from_sim no)
@@
 		(fields_autoplaced yes)
 		(property "Reference" "R3"
-			(at 168.91 111.7599 0)
+			(at 168.91 113.0299 0)
 			(effects
 				(font
@@
 		)
 		(property "Value" "4k7"
-			(at 168.91 114.2999 0)
+			(at 168.91 115.5699 0)
 			(effects
 				(font
@@
 		)
 		(property "Footprint" "Resistor_THT:R_Axial_DIN0204_L3.6mm_D1.6mm_P7.62mm_Horizontal"
-			(at 164.592 113.03 90)
+			(at 164.592 114.3 90)
 			(effects
 				(font
@@
 		)
 		(property "Datasheet" "~"
-			(at 166.37 113.03 0)
+			(at 166.37 114.3 0)
 			(effects
 				(font
@@
 		)
 		(property "Description" "Resistor"
-			(at 166.37 113.03 0)
+			(at 166.37 114.3 0)
 			(effects
 				(font
