File: kicad/pico-gps-spedometer/pico-gps-spedometer.kicad_pcb (KiCad board)
At the start: 2 copper layers, 102 x 57.5 mm, 30 parts, among them J1 Akkumulátor be, J3 uBlox NEO GPS (6M/8M), Q1 PN2222A, Q2 PN2222A, U1 RP2040-ZERO, U2 DS18B20, U3 LM7805_TO220, U4 TFT_320x240

Commit message: Implement code changes to enhance functionality and improve performance
Parts:
- moved REF** 1.25 mm to (148.5, 28.5)
- moved REF** 1.03 mm to (148.5, 79.0)
Changed lines of the file:
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@@
 	(footprint "MountingHole:MountingHole_3.2mm_M3"
 		(layer "F.Cu")
-		(at 147.25 28.5)
+		(at 148.5 28.5)
 		(descr "Mounting Hole 3.2mm, M3, no annular, generated by kicad-footprint-generator mountinghole.py")
 		(tags "mountinghole M3")
@@
 	(footprint "MountingHole:MountingHole_3.2mm_M3"
 		(layer "F.Cu")
-		(at 147.5 78.75)
+		(at 148.5 79)
 		(descr "Mounting Hole 3.2mm, M3, no annular, generated by kicad-footprint-generator mountinghole.py")
 		(tags "mountinghole M3")
